Commit message: 修改mid360参数

File: lightning-lm/urdf/g1.urdf (robot description, URDF)
Before this commit: robot g1_navigation_sensors, 4 links, 3 joints
Joints:
- joint base_to_mid360_joint: origin xyz=0.0002835 0.00003 1.30618 rpy=0 0.04014257279586953 0 -> xyz=0.0002835 0.00003 1.23618 rpy=0 0.04014257279586953 0

Commit message: 完整调通过了

File: lightning-lm/urdf/g1.urdf (robot description, URDF)
Before this commit: robot g1_navigation_sensors, 4 links, 3 joints
Links:
- added link camera_link
- added link d435_link
Joints:
- added joint base_to_d435_joint: type fixed, parent base_link, child d435_link, origin xyz=0.0576235 0.01753 1.24987 rpy=0 0.8307767239493009 0
- added joint d435_to_camera_link_joint: type fixed, parent d435_link, child camera_link, origin xyz=0 0 0 rpy=0 0 0

Commit message: 终于修复了tf的问题

File: lightning-lm/urdf/g1.urdf (robot description, URDF)
Before this commit: robot g1_navigation_sensors, 6 links, 5 joints
Joints:
- joint base_to_mid360_joint: origin xyz=0.0002835 0.00003 1.23618 rpy=0 0.04014257279586953 0 -> xyz=0.0002835 0.00003 1.23618 rpy=0 -0.04014257279586953 0

Commit message: 调试通过

File: lightning-lm/urdf/g1.urdf (robot description, URDF)
Before this commit: robot g1_navigation_sensors, 6 links, 5 joints
Links:
- removed link base_footprint
- removed link base_link
- added link body_link
Joints:
- removed joint base_to_d435_joint
- removed joint base_to_footprint_joint
- removed joint base_to_mid360_joint
- added joint body_to_d435_joint: type fixed, parent body_link, child d435_link, origin xyz=0.0576235 0.01753 1.24987 rpy=0 0.8307767239493009 0
- added joint body_to_mid360_joint: type fixed, parent body_link, child mid360_link, origin xyz=0.0002835 0.00003 1.23618 rpy=0 0.04014257279586953 0
